Commit message: Work on allegro hand grasp

File: configs/urdfs/allegro_hand.urdf (robot description, URDF)
Before this commit: robot allegro_hand_right, 22 links, 21 joints
Links:
- added link intermediate_link_rot_x
- added link intermediate_link_rot_y
- added link intermediate_link_x
- added link intermediate_link_y
- added link intermediate_link_z
Joints:
- removed joint arm_to_world_floating
- added joint rot_x: type revolute, parent intermediate_link_z, child intermediate_link_rot_x, origin xyz=0 0 0 rpy=0 0 0, axis 1 0 0, limit lower=-1000000 upper=1000000 effort=1000 velocity=1
- added joint rot_y: type revolute, parent intermediate_link_rot_x, child intermediate_link_rot_y, origin xyz=0 0 0 rpy=0 0 0, axis 0 1 0, limit lower=-1000000 upper=1000000 effort=1000 velocity=1
- added joint rot_z: type revolute, parent intermediate_link_rot_y, child palm_link, origin xyz=0 0 0 rpy=0 0 0, axis 0 0 1, limit lower=-1000000 upper=1000000 effort=1000 velocity=1
- added joint trans_x: type prismatic, parent world, child intermediate_link_x, origin xyz=0 0 0 rpy=0 0 0, axis 1 0 0, limit lower=-1000000 upper=1000000 effort=1000 velocity=2
- added joint trans_y: type prismatic, parent intermediate_link_x, child intermediate_link_y, origin xyz=0 0 0 rpy=0 0 0, axis 0 1 0, limit lower=-1000000 upper=1000000 effort=1000 velocity=2
- added joint trans_z: type prismatic, parent intermediate_link_y, child intermediate_link_z, origin xyz=0 0 0 rpy=0 0 0, axis 0 0 1, limit lower=-1000000 upper=1000000 effort=1000 velocity=2
- joint joint_11.0_tip: origin xyz=0 0 0.0267 rpy=0 0 0 -> xyz=0 0 0.0407 rpy=0 0 0
- joint joint_15.0_tip: origin xyz=0 0 0.0423 rpy=0 0 0 -> xyz=0 0 0.0563 rpy=0 0 0
- joint joint_3.0_tip: origin xyz=0 0 0.0267 rpy=0 0 0 -> xyz=0 0 0.0407 rpy=0 0 0
- joint joint_7.0_tip: origin xyz=0 0 0.0267 rpy=0 0 0 -> xyz=0 0 0.0407 rpy=0 0 0
